File: schematic/irUsbSender-v1-0-1.kicad_pcb (KiCad board)
At the start: 2 copper layers, 26 x 46.5 mm, 38 parts, among them J1 USB_B_Micro, J2 Conn_01x06_Male, J3 Conn_01x03_Male, J4 Conn_01x02_Male, J5 Conn_01x02_Male, J6 Conn_01x02_Male, J7 Conn_01x08_Male, Q1 IRLML6344, U1 MCP1754-3302E_SOT89, U2 STM32F042K6Tx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

Commit message: Add build workflow. Add cnc milling. Improve doc. Minor fix in schematic. Minor improvement in host program.
Parts:
- C10: value 4,7µF -> 4.7µF
Changed lines of the file:
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@@
   (title_block
     (title IRUSB)
-    (date 2020-11-27)
+    (date 2020-11-28)
     (rev 1.0.1)
     (company "(c) 2020 by Malte Marwedel")
@@
       (effects (font (size 1 1) (thickness 0.15)))
     )
-    (fp_text value 4,7µF (at 0 1.65) (layer F.Fab)
-      (effects (font (size 1 1) (thickness 0.15)))
-    )
+    (fp_text value 4.7µF (at 0 1.65) (layer F.Fab)
+      (effects (font (size 1 1) (thickness 0.15)))
+    )
